Commit message: final commit

File: src/my_robot_description/urdf/my_robot.urdf.xacro (robot description, xacro)
@@ -27,7 +27,9 @@
     <inertial>
       <mass value="5.0"/>
+      <origin xyz="0 0 0" rpy="0 0 0"/>
       <inertia ixx="0.0625" ixy="0.0" ixz="0.0" iyy="0.1104" iyz="0.0" izz="0.1354"/>
     </inertial>
   </link>
+    <!-- Joint connecting base_footprint to base_link -->
   <joint name="base_footprint_to_base_link" type="fixed">
     <parent link="base_footprint"/>
@@ -88,28 +90,4 @@
   </joint>
   <!-- Caster Wheel -->
-  <link name="caster_link">
-    <visual>
-      <geometry>
-        <sphere radius="${caster_radius}"/>
-      </geometry>
-      <material name="gray">
-        <color rgba="0.5 0.5 0.5 1"/>
-      </material>
-    </visual>
-    <collision>
-      <geometry>
-        <sphere radius="${caster_radius}"/>
-      </geometry>
-    </collision>
-    <inertial>
-      <mass value="0.2"/>
-      <inertia ixx="0.0001" ixy="0.0" ixz="0.0" iyy="0.0001" iyz="0.0" izz="0.0001"/>
-    </inertial>
-  </link>
-  <joint name="caster_joint" type="fixed">
-    <parent link="base_link"/>
-    <child link="caster_link"/>
-    <origin xyz="${-chassis_length/2 + caster_radius} 0 ${-chassis_height/2 - caster_radius/2}" rpy="0 0 0"/>
-  </joint>
   <!-- Camera Link -->
   <link name="camera_link">
@@ -129,4 +107,5 @@
     <inertial>
       <mass value="0.1"/>
+      <origin xyz="0 0 0" rpy="0 0 0"/>
       <inertia ixx="0.00001" ixy="0.0" ixz="0.0" iyy="0.00001" iyz="0.0" izz="0.00001"/>
     </inertial>
@@ -135,21 +114,52 @@
     <parent link="base_link"/>
     <child link="camera_link"/>
-    <origin xyz="${chassis_length/2} 0 ${chassis_height/2 + 0.025}" rpy="0 0 0"/>
+    <origin xyz="${chassis_length/2} 0 ${chassis_height/2 + 0.025}" rpy="0 0.2 0"/>
+  </joint>
+  <!-- Counterweight link (balances camera mass) -->
+  <link name="counterweight_link">
+    <visual>
+      <geometry>
+        <box size="0.05 0.05 0.05"/>
+      </geometry>
+      <material name="grey">
+        <color rgba="0.5 0.5 0.5 1"/>
+      </material>
+    </visual>
+    <collision>
+      <geometry>
+        <box size="0.05 0.05 0.05"/>
+      </geometry>
+    </collision>
+    <inertial>
+      <mass value="0.1"/>
+      <origin xyz="0 0 0" rpy="0 0 0"/>
+      <inertia ixx="0.00001" ixy="0.0" ixz="0.0" iyy="0.00001" iyz="0.0" izz="0.00001"/>
+    </inertial>
+  </link>
+  <joint name="counterweight_joint" type="fixed">
+    <parent link="base_link"/>
+    <child link="counterweight_link"/>
+    <origin xyz="${-chassis_length/2} 0 ${chassis_height/2 + 0.025}" rpy="0 0 0"/>
   </joint>
   <!-- Gazebo Differential Drive Plugin -->
   <gazebo>
-    <plugin filename="libgz-sim-diff-drive-system.so" name="gz::sim::systems::DiffDrive">
+    <plugin filename="gz-sim-diff-drive-system" name="gz::sim::systems::DiffDrive">
       <left_joint>left_wheel_joint</left_joint>
       <right_joint>right_wheel_joint</right_joint>
       <wheel_separation>${chassis_width + wheel_width}</wheel_separation>
       <wheel_radius>${wheel_radius}</wheel_radius>
-      <odom_publish_frequency>30</odom_publish_frequency>
-      <topic>/model/my_robot/cmd_vel</topic>
-      <odom_topic>/odometry</odom_topic>
-      <tf_topic>/tf</tf_topic>
+      <odom_publish_frequency>50</odom_publish_frequency>
+      <topic>/cmd_vel</topic>          <!-- Listens to /cmd_vel for movement -->
+      <odom_topic>/odom</odom_topic>   <!-- Publishes odometry messages -->
+      <tf_topic>/tf</tf_topic>         <!-- Publishes the odom->base_footprint transform -->
       <frame_id>odom</frame_id>
       <child_frame_id>base_footprint</child_frame_id>
     </plugin>
-  </gazebo>  <!-- Gazebo Camera Sensor -->
+  </gazebo>
+  <gazebo>
+    <plugin filename="gz-sim-joint-state-publisher-system" name="gz::sim::systems::JointStatePublisher">
+      <topic>/joint_states</topic>
+    </plugin>
+  </gazebo> <!-- Gazebo Camera Sensor -->
   <gazebo reference="camera_link">
     <sensor name="camera" type="camera">
@@ -166,4 +176,5 @@
           <far>100</far>
         </clip>
+        <frame_name>camera_link</frame_name>
       </camera>
       <always_on>1</always_on>
@@ -191,3 +202,6 @@
     <material>Gazebo/Red</material>
   </gazebo>
+  <gazebo reference="counterweight_link">
+    <material>Gazebo/Grey</material>
+  </gazebo>
 </robot>
